Commit message: Friday

File: Hector_ROS_Simulation/hector_description/xacro/gripper.xacro (robot description, xacro)
@@ -2,6 +2,6 @@
 <robot xmlns:xacro="http://www.ros.org/wiki/xacro">
 <xacro:include filename="$(find hector_description)/xacro/arm_transmission.xacro"/>
-    <xacro:macro name="arm" params="name mirror mirror_dae  *origin">
-        <joint name="${name}_twist_joint" type="revolute">
+    <xacro:macro name="gripper" params="name mirror mirror_dae  *origin">
+        <joint name="${name}_gripper_twist_joint" type="revolute">
             <xacro:if value="${(mirror_dae == True)}">
             <origin rpy="0 0 0" xyz="0.0 0.047 0.1725"/>
@@ -11,5 +11,5 @@
             </xacro:if>
             <parent link="trunk"/>
-            <child link="${name}_twist"/>
+            <child link="${name}_gripper_twist"/>
             <axis xyz="0 0 1"/>
             <dynamics damping="${damping}" friction="${friction}"/>
@@ -21,5 +21,5 @@
             </xacro:if>
         </joint>
-        <link name="${name}_twist">
+        <link name="${name}_gripper_twist">
             <visual>
             <origin rpy="0 ${-PI/2.0} 0" xyz="0 0 0"/>
@@ -49,5 +49,15 @@
             </inertial> -->
         </link>
-        <joint name="${name}_shoulder_joint" type="revolute">
+        <transmission name="${name}_gripper_twist_tran">
+            <type>transmission_interface/SimpleTransmission</type>
+            <joint name="${name}_gripper_twist_joint">
+            <hardwareInterface>hardware_interface/EffortJointInterface</hardwareInterface>
+            </joint>
+            <actuator name="${name}_gripper_twist_motor">
+            <hardwareInterface>hardware_interface/EffortJointInterface</hardwareInterface>
+            <mechanicalReduction>1</mechanicalReduction>
+            </actuator>
+        </transmission>
+        <joint name="${name}_gripper_shoulder_joint" type="revolute">
             <xacro:if value="${(mirror_dae == True)}">
             <origin rpy="0 0 0" xyz="0.0 0.0723 0.0"/>
@@ -56,11 +66,11 @@
             <origin rpy="0 0 0" xyz="0.0 -0.0723 0.0"/>
             </xacro:if>
-            <parent link="${name}_twist"/>
-            <child link="${name}_shoulder"/>
+            <parent link="${name}_gripper_twist"/>
+            <child link="${name}_gripper_shoulder"/>
             <axis xyz="0 1 0"/>
-            <dynamics damping="1" friction="1"/>
+            <dynamics damping="$1" friction="$1"/>
             <limit effort="${shoulder_torque_max}" velocity="${shoulder_velocity_max}" lower="${shoulder_min}" upper="${shoulder_max}"/>
         </joint>
-        <link name="${name}_shoulder">
+        <link name="${name}_gripper_shoulder">
             <visual>
             <origin rpy="0 0 0" xyz="0 0 0"/>
@@ -92,13 +102,23 @@
             </inertial>
         </link>
-        <joint name="${name}_elbow_joint" type="revolute">
+        <transmission name="${name}_gripper_shoulder_tran">
+            <type>transmission_interface/SimpleTransmission</type>
+            <joint name="${name}_gripper_shoulder_joint">
+            <hardwareInterface>hardware_interface/EffortJointInterface</hardwareInterface>
+            </joint>
+            <actuator name="${name}_gripper_shoulder_motor">
+            <hardwareInterface>hardware_interface/EffortJointInterface</hardwareInterface>
+            <mechanicalReduction>1</mechanicalReduction>
+            </actuator>
+        </transmission>
+        <joint name="${name}_gripper_elbow_joint" type="revolute">
             <origin rpy="0 -1.5 0" xyz="0.0 0.0 -0.205"/>
-            <parent link="${name}_shoulder"/>
-            <child link="${name}_elbow"/>
+            <parent link="${name}_gripper_shoulder"/>
+            <child link="${name}_gripper_elbow"/>
             <axis xyz="0 1 0"/>
             <dynamics damping="1" friction="1"/>
             <limit effort="${elbow_torque_max}" velocity="${elbow_velocity_max}" lower="${elbow_min}" upper="${elbow_max}"/>
         </joint>
-        <link name="${name}_elbow">
+        <link name="${name}_gripper_elbow">
             <visual>
             <origin rpy="0 0 0" xyz="0 0 0"/>
@@ -123,5 +143,14 @@
             </inertial>
         </link>
-        <xacro:arm_transmission name="${name}"/>
+        <transmission name="${name}_gripper_elbow_tran">
+            <type>transmission_interface/SimpleTransmission</type>
+            <joint name="${name}_gripper_elbow_joint">
+            <hardwareInterface>hardware_interface/EffortJointInterface</hardwareInterface>
+            </joint>
+            <actuator name="${name}_gripper_twist_motor">
+            <hardwareInterface>hardware_interface/EffortJointInterface</hardwareInterface>
+            <mechanicalReduction>1</mechanicalReduction>
+            </actuator>
+        </transmission>
         <!-- ros control plugin with mimic-->
         <xacro:macro name="mimic_joint_plugin_gazebo" params="parent_joint mimic_joint has_pid:=false multiplier:=-1.0 offset:=0 sensitiveness:=0.0 max_effort:=200 robot_namespace:='/hector_gazebo'">
@@ -143,5 +172,5 @@
             </gazebo>
         </xacro:macro>
-        <xacro:mimic_joint_plugin_gazebo  parent_joint="R_elbow_joint" mimic_joint="L_elbow_joint"
+        <xacro:mimic_joint_plugin_gazebo  parent_joint="R_gripper_elbow_joint" mimic_joint="L_gripper_elbow_joint"
                                             has_pid="false" multiplier="-1.0" max_effort="200" />
         <gazebo>
